File: hardware/PGTN034_quantizer_mki_controls.sch (EAGLE design)
At the start: 114 parts, among them Q1 2N3904SOT23, Q2 2N3904SOT23, Q3 2N3904SOT23, Q4 2N3904SOT23, SW1 ENCODER_SW1-PEC12, SW2 ENCODER_SW1-PEC12

Commit message: set offset when changing scale
Connections:
- new net N$4: 0_RX.3, TFT1.RES
- new net N$57: 1_TX.3, U$2.CS/SS
Other:
- moved on the sheet: 0_RX, 1_TX
Changed lines of the file:
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@@
 <attribute name="NAME" x="47.244" y="1.524" size="1.778" layer="96"/>
 </instance>
-<instance part="1_TX" gate="HEADER" x="2.54" y="50.8" smashed="yes">
-<attribute name="NAME" x="-11.176" y="49.784" size="1.778" layer="96"/>
-</instance>
-<instance part="0_RX" gate="HEADER" x="2.54" y="53.34" smashed="yes">
-<attribute name="NAME" x="-11.176" y="52.324" size="1.778" layer="96"/>
+<instance part="1_TX" gate="HEADER" x="58.42" y="104.14" smashed="yes">
+<attribute name="NAME" x="44.704" y="103.124" size="1.778" layer="96"/>
+</instance>
+<instance part="0_RX" gate="HEADER" x="60.96" y="134.62" smashed="yes">
+<attribute name="NAME" x="47.244" y="133.604" size="1.778" layer="96"/>
 </instance>
 <instance part="CV7_" gate="HEADER" x="2.54" y="-137.16" smashed="yes">
@@
 </segment>
 </net>
+<net name="N$4" class="0">
+<segment>
+<pinref part="TFT1" gate="G$1" pin="RES"/>
+<wire x1="76.2" y1="134.62" x2="63.5" y2="134.62" width="0.1524" layer="91"/>
+<pinref part="0_RX" gate="HEADER" pin="3"/>
+</segment>
+</net>
+<net name="N$57" class="0">
+<segment>
+<pinref part="1_TX" gate="HEADER" pin="3"/>
+<pinref part="U$2" gate="G$1" pin="CS/SS"/>
+<wire x1="60.96" y1="104.14" x2="76.2" y2="104.14" width="0.1524" layer="91"/>
+</segment>
+</net>
